File: Pr0Board_Cheap/Hardware/pr0board_key.brd (EAGLE design)
At the start: 86.4 x 49.5 mm, 29 parts, among them M1 DSA_KEYCAP, M2 DSA_KEYCAP, M3 DSA_KEYCAP, M4 DSA_KEYCAP, M5 DSA_KEYCAP, M6 DSA_KEYCAP, M7 DSA_KEYCAP, M8 DSA_KEYCAP

Commit message: Cleanup
Parts:
- removed LED10, LED11, LED9: WS2812B3535, adafruit:LED3535
- added LED1, LED2, LED3: WS2812B3535, adafruit:LED3535
- moved LED4 57.1 mm to (71.8, 39.6)
- moved LED8 57.1 mm to (71.8, 9.92)
- moved LED5 35.3 mm to (14.6, 9.92)
- moved LED6 35.3 mm to (33.7, 9.92)
- moved LED7 35.3 mm to (52.7, 9.92)
Connections:
- removed net N$13 (its old number): LED8.2, LED9.4
- removed net N$14 (its old number): LED10.4, LED9.2
- new net N$10: LED3.2, LED4.4
- new net N$9: LED2.2, LED3.4
- net DODI: now also LED4.2, LED5.4; no longer LED7.2, LED8.4
- net GND: now also LED1.3, LED2.3, LED3.3; no longer LED10.3, LED11.3, LED9.3
- net N$15: now also LED7.2, LED8.4; no longer LED10.2, LED11.4
- net N$8: now also LED1.2, LED2.4; no longer LED4.2, LED5.4
- net WS2812BDI: now also LED1.4; no longer LED4.4
- net WS2812BDO: now also LED8.2; no longer LED11.2
- net WSVCC: now also LED1.1, LED2.1, LED3.1; no longer LED10.1, LED11.1, LED9.1
Routing:
- net N$14 (its old number): track 26.5 -> 0.00 mm, vias 2 -> 0
- net N$13 (its old number): track 24.1 -> 0.00 mm
- net N$10: track 0.00 -> 22.9 mm
- net N$9: track 0.00 -> 22.9 mm
- net N$14: track 22.9 -> 26.5 mm, vias 0 -> 2
- net N$13: track 22.9 -> 24.1 mm
Changed lines of the file:
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@@
 <attribute name="VALUE" x="64.77" y="0.889" size="1.27" layer="28" ratio="10" rot="MR0"/>
 </element>
-<element name="LED4" library="adafruit" package="LED3535" override_package3d_urn="urn:adsk.eagle:package:22982386/2" override_package_urn="urn:adsk.eagle:footprint:22982387/1" override_locally_modified="yes" value="WS2812B3535" x="14.605" y="39.608125" smashed="yes" rot="R270">
+<element name="LED1" library="adafruit" package="LED3535" override_package3d_urn="urn:adsk.eagle:package:22982386/2" override_package_urn="urn:adsk.eagle:footprint:22982387/1" override_locally_modified="yes" value="WS2812B3535" x="14.605" y="39.608125" smashed="yes" rot="R270">
 <attribute name="VALUE" x="12.065" y="41.386125" size="0.4064" layer="27" ratio="10" rot="R270"/>
 </element>
-<element name="LED5" library="adafruit" package="LED3535" override_package3d_urn="urn:adsk.eagle:package:22982386/2" override_package_urn="urn:adsk.eagle:footprint:22982387/1" override_locally_modified="yes" value="WS2812B3535" x="33.655" y="39.608125" smashed="yes" rot="R270">
+<element name="LED2" library="adafruit" package="LED3535" override_package3d_urn="urn:adsk.eagle:package:22982386/2" override_package_urn="urn:adsk.eagle:footprint:22982387/1" override_locally_modified="yes" value="WS2812B3535" x="33.655" y="39.608125" smashed="yes" rot="R270">
 <attribute name="VALUE" x="31.115" y="41.386125" size="0.4064" layer="27" ratio="10" rot="R270"/>
 </element>
-<element name="LED6" library="adafruit" package="LED3535" override_package3d_urn="urn:adsk.eagle:package:22982386/2" override_package_urn="urn:adsk.eagle:footprint:22982387/1" override_locally_modified="yes" value="WS2812B3535" x="52.705" y="39.608125" smashed="yes" rot="R270">
+<element name="LED3" library="adafruit" package="LED3535" override_package3d_urn="urn:adsk.eagle:package:22982386/2" override_package_urn="urn:adsk.eagle:footprint:22982387/1" override_locally_modified="yes" value="WS2812B3535" x="52.705" y="39.608125" smashed="yes" rot="R270">
 <attribute name="VALUE" x="50.165" y="41.386125" size="0.4064" layer="27" ratio="10" rot="R270"/>
 </element>
-<element name="LED7" library="adafruit" package="LED3535" override_package3d_urn="urn:adsk.eagle:package:22982386/2" override_package_urn="urn:adsk.eagle:footprint:22982387/1" override_locally_modified="yes" value="WS2812B3535" x="71.755" y="39.608125" smashed="yes" rot="R270">
+<element name="LED4" library="adafruit" package="LED3535" override_package3d_urn="urn:adsk.eagle:package:22982386/2" override_package_urn="urn:adsk.eagle:footprint:22982387/1" override_locally_modified="yes" value="WS2812B3535" x="71.755" y="39.608125" smashed="yes" rot="R270">
 <attribute name="VALUE" x="69.215" y="41.386125" size="0.4064" layer="27" ratio="10" rot="R270"/>
 </element>
-<element name="LED8" library="adafruit" package="LED3535" override_package3d_urn="urn:adsk.eagle:package:22982386/2" override_package_urn="urn:adsk.eagle:footprint:22982387/1" override_locally_modified="yes" value="WS2812B3535" x="14.605" y="9.921875" smashed="yes" rot="R270">
+<element name="LED5" library="adafruit" package="LED3535" override_package3d_urn="urn:adsk.eagle:package:22982386/2" override_package_urn="urn:adsk.eagle:footprint:22982387/1" override_locally_modified="yes" value="WS2812B3535" x="14.605" y="9.921875" smashed="yes" rot="R270">
 <attribute name="VALUE" x="12.065" y="11.699875" size="0.4064" layer="27" ratio="10" rot="R270"/>
 </element>
-<element name="LED9" library="adafruit" package="LED3535" override_package3d_urn="urn:adsk.eagle:package:22982386/2" override_package_urn="urn:adsk.eagle:footprint:22982387/1" override_locally_modified="yes" value="WS2812B3535" x="33.655" y="9.921875" smashed="yes" rot="R270">
+<element name="LED6" library="adafruit" package="LED3535" override_package3d_urn="urn:adsk.eagle:package:22982386/2" override_package_urn="urn:adsk.eagle:footprint:22982387/1" override_locally_modified="yes" value="WS2812B3535" x="33.655" y="9.921875" smashed="yes" rot="R270">
 <attribute name="VALUE" x="31.115" y="11.699875" size="0.4064" layer="27" ratio="10" rot="R270"/>
 </element>
-<element name="LED10" library="adafruit" package="LED3535" override_package3d_urn="urn:adsk.eagle:package:22982386/2" override_package_urn="urn:adsk.eagle:footprint:22982387/1" override_locally_modified="yes" value="WS2812B3535" x="52.705" y="9.921875" smashed="yes" rot="R270">
+<element name="LED7" library="adafruit" package="LED3535" override_package3d_urn="urn:adsk.eagle:package:22982386/2" override_package_urn="urn:adsk.eagle:footprint:22982387/1" override_locally_modified="yes" value="WS2812B3535" x="52.705" y="9.921875" smashed="yes" rot="R270">
 <attribute name="VALUE" x="50.165" y="11.699875" size="0.4064" layer="27" ratio="10" rot="R270"/>
 </element>
-<element name="LED11" library="adafruit" package="LED3535" override_package3d_urn="urn:adsk.eagle:package:22982386/2" override_package_urn="urn:adsk.eagle:footprint:22982387/1" override_locally_modified="yes" value="WS2812B3535" x="71.755" y="9.921875" smashed="yes" rot="R270">
+<element name="LED8" library="adafruit" package="LED3535" override_package3d_urn="urn:adsk.eagle:package:22982386/2" override_package_urn="urn:adsk.eagle:footprint:22982387/1" override_locally_modified="yes" value="WS2812B3535" x="71.755" y="9.921875" smashed="yes" rot="R270">
 <attribute name="VALUE" x="69.215" y="11.699875" size="0.4064" layer="27" ratio="10" rot="R270"/>
 </element>
@@
 <contactref element="S1" pad="L2"/>
 <contactref element="SV3" pad="1"/>
+<contactref element="LED1" pad="3"/>
+<contactref element="LED2" pad="3"/>
+<contactref element="LED3" pad="3"/>
 <contactref element="LED4" pad="3"/>
 <contactref element="LED5" pad="3"/>
@@
 <contactref element="LED7" pad="3"/>
 <contactref element="LED8" pad="3"/>
-<contactref element="LED9" pad="3"/>
-<contactref element="LED10" pad="3"/>
-<contactref element="LED11" pad="3"/>
 <contactref element="S2" pad="S2"/>
 <contactref element="S2" pad="L2"/>
@@
 <signal name="WS2812BDI">
 <contactref element="SV1" pad="5"/>
-<contactref element="LED4" pad="4"/>
+<contactref element="LED1" pad="4"/>
 <wire x1="13.02" y1="40.394575" x2="12.6827" y2="40.731875" width="0.3048" layer="1"/>
 <wire x1="12.6827" y1="40.731875" x2="12.6827" y2="42.460625" width="0.3048" layer="1"/>
@@
 <signal name="WS2812BDO">
 <contactref element="SV4" pad="1"/>
-<contactref element="LED11" pad="2"/>
+<contactref element="LED8" pad="2"/>
 <wire x1="70.88" y1="11.671875" x2="69.0525" y2="11.671875" width="0.3048" layer="1"/>
 <wire x1="69.0525" y1="11.671875" x2="68.659375" y2="12.065" width="0.3048" layer="1"/>
@@
 </signal>
 <signal name="N$8">
-<contactref element="LED4" pad="2"/>
-<contactref element="LED5" pad="4"/>
+<contactref element="LED1" pad="2"/>
+<contactref element="LED2" pad="4"/>
 <wire x1="32.9409" y1="40.408175" x2="33.6613" y2="39.687775" width="0.3048" layer="1"/>
 <wire x1="13.73" y1="41.358125" x2="14.67995" y2="40.408175" width="0.3048" layer="1"/>
@@
 </signal>
 <signal name="N$9">
-<contactref element="LED5" pad="2"/>
-<contactref element="LED6" pad="4"/>
+<contactref element="LED2" pad="2"/>
+<contactref element="LED3" pad="4"/>
 <wire x1="51.9909" y1="40.408175" x2="52.7113" y2="39.687775" width="0.3048" layer="1"/>
 <wire x1="52.7113" y1="39.687775" x2="52.7113" y2="38.726825" width="0.3048" layer="1"/>
@@
 </signal>
 <signal name="N$10">
-<contactref element="LED6" pad="2"/>
-<contactref element="LED7" pad="4"/>
+<contactref element="LED3" pad="2"/>
+<contactref element="LED4" pad="4"/>
 <wire x1="71.120275" y1="40.408175" x2="71.7613" y2="39.76715" width="0.3048" layer="1"/>
 <wire x1="71.7613" y1="39.76715" x2="71.7613" y2="38.726825" width="0.3048" layer="1"/>
@@
 </signal>
 <signal name="N$13">
-<contactref element="LED8" pad="2"/>
-<contactref element="LED9" pad="4"/>
+<contactref element="LED5" pad="2"/>
+<contactref element="LED6" pad="4"/>
 <wire x1="14.5987" y1="9.683475" x2="15.16035" y2="9.121825" width="0.3048" layer="1"/>
 <wire x1="32.07" y1="6.890825" x2="33.49" y2="6.890825" width="0.3048" layer="1"/>
@@
 </signal>
 <signal name="N$14">
-<contactref element="LED9" pad="2"/>
-<contactref element="LED10" pad="4"/>
+<contactref element="LED6" pad="2"/>
+<contactref element="LED7" pad="4"/>
 <wire x1="32.78" y1="11.671875" x2="31.595" y2="11.671875" width="0.3048" layer="1"/>
 <wire x1="31.595" y1="11.671875" x2="31.59125" y2="11.668125" width="0.3048" layer="1"/>
@@
 </signal>
 <signal name="N$15">
-<contactref element="LED10" pad="2"/>
-<contactref element="LED11" pad="4"/>
+<contactref element="LED7" pad="2"/>
+<contactref element="LED8" pad="4"/>
 <wire x1="51.83" y1="11.671875" x2="50.80375" y2="11.671875" width="0.3048" layer="1"/>
 <wire x1="50.80375" y1="11.671875" x2="50.8" y2="11.668125" width="0.3048" layer="1"/>
@@
 </signal>
 <signal name="WSVCC">
+<contactref element="LED1" pad="1"/>
+<contactref element="LED2" pad="1"/>
+<contactref element="LED3" pad="1"/>
 <contactref element="LED4" pad="1"/>
 <contactref element="LED5" pad="1"/>
@@
 <contactref element="LED7" pad="1"/>
 <contactref element="LED8" pad="1"/>
-<contactref element="LED9" pad="1"/>
-<contactref element="LED10" pad="1"/>
-<contactref element="LED11" pad="1"/>
 <contactref element="SV2" pad="1"/>
 <wire x1="32.149375" y1="42.5598" x2="33.410625" y2="42.5598" width="0.3048" layer="1"/>
@@
 </signal>
 <signal name="DODI">
-<contactref element="LED8" pad="4"/>
-<contactref element="LED7" pad="2"/>
+<contactref element="LED5" pad="4"/>
+<contactref element="LED4" pad="2"/>
 <wire x1="72.07875" y1="40.553325" x2="72.0798" y2="40.553325" width="0.3048" layer="1"/>
 <wire x1="72.0798" y1="40.553325" x2="72.23125" y2="40.401875" width="0.3048" layer="1"/>
