File: Pr0Board_Cheap/Hardware/pr0board_key.sch (EAGLE design)
At the start: 29 parts, among them M1 DSA_KEYCAP, M2 DSA_KEYCAP, M3 DSA_KEYCAP, M4 DSA_KEYCAP, M5 DSA_KEYCAP, M6 DSA_KEYCAP, M7 DSA_KEYCAP, M8 DSA_KEYCAP

Commit message: Cleanup
Parts:
- removed LED10, LED11, LED9: WS2812B3535, adafruit:WS2812B3535
- added LED1, LED2, LED3: WS2812B3535, adafruit:WS2812B3535
Connections:
- removed net N$13 (its old number): LED8.DO, LED9.DI
- removed net N$14 (its old number): LED10.DI, LED9.DO
- new net N$10: LED3.DO, LED4.DI
- new net N$9: LED2.DO, LED3.DI
- net DODI: now also LED4.DO, LED5.DI; no longer LED7.DO, LED8.DI
- net GND: now also LED1.GND, LED2.GND, LED3.GND; no longer LED10.GND, LED11.GND, LED9.GND
- net N$15: now also LED7.DO, LED8.DI; no longer LED10.DO, LED11.DI
- net N$8: now also LED1.DO, LED2.DI; no longer LED4.DO, LED5.DI
- net WS2812BDI: now also LED1.DI; no longer LED4.DI
- net WS2812BDO: now also LED8.DO; no longer LED11.DO
- net WSVCC: now also LED1.VDD, LED2.VDD, LED3.VDD; no longer LED10.VDD, LED11.VDD, LED9.VDD
