File: Pr0Board_Cheap/Hardware/pr0board_main.sch (EAGLE design)
At the start: 20 parts, among them Q1 MMBTA56-SOT23

Commit message: Cleanup
Parts:
- Q1: value MMBTA56-SOT23 -> NC
- R10: value 22R -> NC
- R3, R5, R6: value 330R -> 1k
- R9: value 1K -> NC
- renumbered B1 to U1
