File: Pr0board_Lite/Hardware/eagle/Pr0board_Lite_Main.brd (EAGLE design)
At the start: 97 x 45 mm, 42 parts, among them J2 10118194-0001LF, J3 TYPE-C-31-M-12

Commit message: fw & bootloader
Routing:
- net VCC: track 234.8 -> 238.0 mm
- net COL4: track 91.4 -> 93.0 mm
- net PB0: track 47.3 -> 48.3 mm
- net N$4: track 36.6 -> 37.7 mm
Other:
- board text added: "v1.1"
- board text removed: "v1.0"
Changed lines of the file:
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@@
 <text x="5" y="0.5" size="1.778" layer="25" font="vector">&gt;_ Pr0Board Lite MX</text>
 <text x="67.5" y="1" size="1.778" layer="25" font="vector">ripper121.com</text>
-<text x="24.5" y="41.5" size="1.778" layer="25" font="vector">v1.0</text>
+<text x="24.5" y="41.5" size="1.778" layer="25" font="vector">v1.1</text>
 <text x="61" y="41.5" size="1.778" layer="25" font="vector">Unknown23</text>
 </plain>
@@
 <wire x1="46" y1="40.8" x2="44.530625" y2="40.8" width="0.3048" layer="1"/>
 <wire x1="44.530625" y1="40.8" x2="44.529375" y2="40.79875" width="0.3048" layer="1"/>
-<via x="6.82625" y="36.274375" extent="1-16" drill="0.35"/>
+<via x="6.19125" y="35.480625" extent="1-16" drill="0.35"/>
 <via x="9.36625" y="36.274375" extent="1-16" drill="0.35"/>
 <contactref element="J3" pad="S3"/>
@@
 <wire x1="84.61486875" y1="37.99" x2="85.59426875" y2="38.9694" width="0.3048" layer="1"/>
 <wire x1="86.62573125" y1="38.9694" x2="87.60513125" y2="37.99" width="0.3048" layer="1"/>
-<wire x1="1.870075" y1="10.7748875" x2="1.870075" y2="32.24520625" width="0.3048" layer="1"/>
+<wire x1="1.870075" y1="8.1555125" x2="1.870075" y2="32.24520625" width="0.3048" layer="1"/>
 <wire x1="1.870075" y1="32.24520625" x2="8.67736875" y2="39.0525" width="0.3048" layer="1"/>
-<wire x1="9.11" y1="5.01" x2="7.6349625" y2="5.01" width="0.3048" layer="1"/>
-<wire x1="7.6349625" y1="5.01" x2="1.870075" y2="10.7748875" width="0.3048" layer="1"/>
+<wire x1="9.11" y1="5.01" x2="5.0155875" y2="5.01" width="0.3048" layer="1"/>
+<wire x1="5.0155875" y1="5.01" x2="1.870075" y2="8.1555125" width="0.3048" layer="1"/>
 <wire x1="8.67736875" y1="39.0525" x2="10.00125" y2="39.0525" width="0.3048" layer="1"/>
 <wire x1="10.00125" y1="39.0525" x2="10.89" y2="38.16375" width="0.3048" layer="1"/>
@@
 <wire x1="56.052475" y1="33.90685" x2="62.07125" y2="39.925625" width="0.3048" layer="1"/>
 <wire x1="62.07125" y1="39.925625" x2="67.706875" y2="39.925625" width="0.3048" layer="1"/>
-<wire x1="67.11" y1="5.01" x2="60.16625" y2="11.95375" width="0.3048" layer="1"/>
-<wire x1="60.16625" y1="11.95375" x2="60.16625" y2="16.98625" width="0.3048" layer="1"/>
+<wire x1="67.11" y1="5.01" x2="64.2525" y2="5.01" width="0.3048" layer="1"/>
+<wire x1="64.2525" y1="5.01" x2="60.16625" y2="9.09625" width="0.3048" layer="1"/>
+<wire x1="60.16625" y1="9.09625" x2="60.16625" y2="16.98625" width="0.3048" layer="1"/>
 <via x="60.16625" y="16.98625" extent="1-16" drill="0.35"/>
 <wire x1="60.16625" y1="16.98625" x2="60.16625" y2="21.715625" width="0.3048" layer="16"/>
@@
 <contactref element="LED2" pad="4"/>
 <via x="37.08185" y="10.398125" extent="1-16" drill="0.35"/>
-<wire x1="37.08185" y1="31.29063125" x2="33.86248125" y2="34.51" width="0.3048" layer="1"/>
-<wire x1="29.89" y1="34.51" x2="33.86248125" y2="34.51" width="0.3048" layer="1"/>
-<wire x1="37.08185" y1="31.29063125" x2="37.08185" y2="10.398125" width="0.3048" layer="1"/>
+<wire x1="37.08185" y1="33.03688125" x2="35.60873125" y2="34.51" width="0.3048" layer="1"/>
+<wire x1="29.89" y1="34.51" x2="35.60873125" y2="34.51" width="0.3048" layer="1"/>
+<wire x1="37.08185" y1="33.03688125" x2="37.08185" y2="10.398125" width="0.3048" layer="1"/>
 <wire x1="37.08185" y1="10.398125" x2="38.5106" y2="8.969375" width="0.3048" layer="16"/>
 <wire x1="38.5106" y1="8.969375" x2="52.22875" y2="8.969375" width="0.3048" layer="16"/>
@@
 <contactref element="LED1" pad="2"/>
 <contactref element="LED3" pad="4"/>
-<wire x1="9.11" y1="37.99" x2="9.11" y2="37.751875" width="0.3048" layer="1"/>
-<wire x1="9.11" y1="37.751875" x2="2.936875" y2="31.57875" width="0.3048" layer="1"/>
-<wire x1="5.63875" y1="8.49" x2="9.11" y2="8.49" width="0.3048" layer="1"/>
-<wire x1="2.936875" y1="31.57875" x2="2.936875" y2="11.191875" width="0.3048" layer="1"/>
-<wire x1="2.936875" y1="11.191875" x2="5.63875" y2="8.49" width="0.3048" layer="1"/>
+<wire x1="9.11" y1="37.99" x2="7.284375" y2="36.164375" width="0.3048" layer="1"/>
+<wire x1="7.284375" y1="36.164375" x2="7.284375" y2="28.226875" width="0.3048" layer="1"/>
+<wire x1="7.284375" y1="28.226875" x2="2.936875" y2="23.879375" width="0.3048" layer="1"/>
+<wire x1="3.8925" y1="8.49" x2="9.11" y2="8.49" width="0.3048" layer="1"/>
+<wire x1="2.936875" y1="23.879375" x2="2.936875" y2="9.445625" width="0.3048" layer="1"/>
+<wire x1="2.936875" y1="9.445625" x2="3.8925" y2="8.49" width="0.3048" layer="1"/>
 </signal>
 <signal name="N$10">
@@
 <contactref element="R8" pad="2"/>
 <contactref element="S10" pad="C"/>
-<wire x1="9.68375" y1="1.27" x2="53.101875" y2="1.27" width="0.3048" layer="1"/>
+<wire x1="7.064375" y1="1.27" x2="53.101875" y2="1.27" width="0.3048" layer="1"/>
 <wire x1="53.101875" y1="1.27" x2="53.95" y2="2.118125" width="0.3048" layer="1"/>
 <wire x1="53.95" y1="2.118125" x2="53.95" y2="3" width="0.3048" layer="1"/>
-<wire x1="0.99695" y1="32.443825" x2="0.99695" y2="9.9568" width="0.3048" layer="1"/>
-<wire x1="0.99695" y1="9.9568" x2="9.68375" y2="1.27" width="0.3048" layer="1"/>
+<wire x1="0.99695" y1="32.443825" x2="0.99695" y2="7.337425" width="0.3048" layer="1"/>
+<wire x1="0.99695" y1="7.337425" x2="7.064375" y2="1.27" width="0.3048" layer="1"/>
 <wire x1="9" y1="40.05" x2="8.603125" y2="40.05" width="0.3048" layer="1"/>
 <wire x1="8.603125" y1="40.05" x2="0.99695" y2="32.443825" width="0.3048" layer="1"/>
